Commit message: ACTUALLY committing the right file, URDF second attempt

File: robot_calibration/urdf/simple_2link_arm.urdf (robot description, URDF)
Before this commit: robot pino_first_try, 3 links, 2 joints
Links:
- removed link arm_1
- removed link arm_2
- added link link_1; visual box size=1.8 0.02 0.1
- added link link_2; visual box size=1 0.02 0.1
Joints:
- removed joint arm_1_to_arm_2
- removed joint base_to_arm_1
- added joint base_to_link_1: type revolute, parent base_link, child link_1, origin xyz=0.0 0.0 0.0, axis 0 1 0, limit lower=0.0 upper=6.28 effort=1000.0 velocity=50.0
- added joint link_1_to_link_2: type revolute, parent link_1, child link_2, origin xyz=1.8 0 0, axis 0 1 0, limit lower=0.0 upper=6.28 effort=1000.0 velocity=50.0

Commit message: Addressed issues of previous PR

File: robot_calibration/urdf/simple_2link_arm.urdf (robot description, URDF)
Before this commit: robot pino_first_try, 3 links, 2 joints
Joints:
- joint base_to_link_1: limit lower=0.0 upper=6.28 effort=1000.0 velocity=50.0 -> lower=0.0 upper=6.2831853 effort=1000.0 velocity=50.0
- joint link_1_to_link_2: limit lower=0.0 upper=6.28 effort=1000.0 velocity=50.0 -> lower=0.0 upper=6.2831853 effort=1000.0 velocity=50.0

Commit message: Fixing sign rotation convention

File: robot_calibration/urdf/simple_2link_arm.urdf (robot description, URDF)
Before this commit: robot pino_milestone1_robot, 3 links, 2 joints
Joints:
- joint base_to_link_1: axis 0 1 0 -> 0 -1 0
- joint link_1_to_link_2: axis 0 1 0 -> 0 -1 0
